File: Micro-Mouse PCB Board/Design_1.kicad_sch (KiCad schematic)
At the start: 0 parts

Commit message: Latest Files
v1.0 of Micro-Mouse PCB Design
Other:
- added sheet 2x16 Connector Pins (Connector_Pins_PowerSystem.kicad_sch)
- added sheet Battery (Battery.kicad_sch)
- added sheet Battery Charger - BQ24090 (Battery_Charger.kicad_sch)
- added sheet Battery Charger - BQ24091 (Battery_Charger.kicad_sch)
- added sheet Battery Monitor - 3V3 Battery Input (Battery_Monitor.kicad_sch)
- added sheet Battery Monitor - 9V USB-C Input (Battery_Monitor.kicad_sch)
- added sheet Buck Converter (Buck_Converter.kicad_sch)
- added sheet Final Design 1 (Final_Design_1.kicad_sch)
- added sheet Switch Circuit (IC) MAX869L (Switch_Circuit.kicad_sch)
- added sheet Switch Circuit Slide (Switch_Circuit_Slide.kicad_sch)
- company: (none) -> University of Cape Town
- title: (none) -> EEE3088F Project PCB Design
