File: Micro-Mouse PCB Board/Micro-Mouse PCB Board.kicad_sch (KiCad schematic)
At the start: 0 parts

Commit message: Latest Files
v1.0 of Micro-Mouse PCB Design
Other:
- removed sheet Microcontroller
- removed sheet Sensing System
- company: (none) -> University of Cape Town
- title: (none) -> EEE3088F Project PCB Design
