File: Micro-Mouse PCB Board/Microcontroller.sch.kicad_sch (KiCad schematic)
At the start: 1 part, among them U1 STM32L476VGTx

Commit message: Latest Files
v1.0 of Micro-Mouse PCB Design
Other:
- company: (none) -> University of Cape Town
- title: (none) -> EEE3088F Project PCB Design
Changed lines of the file:
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@@
 	(generator_version "9.0")
 	(paper "A4")
+	(title_block
+		(title "EEE3088F Project PCB Design")
+		(date "2025-03-24")
+		(company "University of Cape Town")
+		(comment 3 "         Emmanual Basua")
+		(comment 4 "Authors: Nejdet Demirtas")
+	)
 	(hierarchical_label "A14"
 		(shape input)
